Commit message: June 24th-2

File: 105_MUJOCO_basic/107_jdcobot100_MUJOCO_load/answer/jdcobot100.urdf (robot description, URDF)
Before this commit: robot jdcobot100_urdf, 5 links, 4 joints
Links:
- link arm_1_sub_asssembly: geometry collision mesh filename=arm_1.stl; collision mesh filename=sg90___micro_servo_9g___tower_pro_1_pe_a.stl
- link arm_2_sub_asssembly_copy_1: geometry collision mesh filename=arm_1.stl; collision mesh filename=sg90___micro_servo_9g___tower_pro_1_pe_a.stl
- link base_sub_assembly: geometry collision mesh filename=base.stl; collision mesh filename=base_link.stl
- link end_arm_sub_assembly: geometry collision mesh filename=arm_end.stl; collision mesh filename=sg90___micro_servo_9g___tower_pro_3_pe_a.stl
- link shoulder_sub_assembly: geometry collision mesh filename=sg90___micro_servo_9g___tower_pro_1_pe_a.stl; collision mesh filename=sg90___micro_servo_9g___tower_pro_1_pe_a__10.stl
